File: classd-amp.kicad_pcb (KiCad board)
At the start: 2 copper layers, 180 x 133.3 mm, 168 parts, among them J1 POWER, J2 Conn_Coaxial_x2, J3 LEFT, J4 RIGHT, J5 POWER, Q1 IRF540N, Q10 IRF540N, Q11 IRF540N, Q12 2N3906, Q2 IRF540N, Q3 IRF540N, Q4 IRF540N, Q5 2N3906, Q6 2N3904, Q7 2N3904, Q8 IRF540N, Q9 IRF540N, U1 TL072, U10 TL072, U11 TL072, U12 LT1016, U13 IR2184, U14 IR2184, U2 TL072, U3 NE555P, U4 LT1016, U5 IR2184, U6 IR2184, U7 LM7812_TO220, U8 LM7805_TO220, U9 LM358

Commit message: Ver 1.1
Parts:
- added D15: SB140, Diode_THT:D_DO-41_SOD81_P10.16mm_Horizontal, F.Cu at (90.7, 75.4)
- added D16: SB140, Diode_THT:D_DO-41_SOD81_P10.16mm_Horizontal, F.Cu at (108.2, 93.7)
- added D17: SB140, Diode_THT:D_DO-41_SOD81_P10.16mm_Horizontal, F.Cu at (109.0, 76.7)
- added D18: SB140, Diode_THT:D_DO-41_SOD81_P10.16mm_Horizontal, F.Cu at (115.6, 76.7)
- added D19: SB140, Diode_THT:D_DO-41_SOD81_P10.16mm_Horizontal, F.Cu at (102.1, 128.3)
- added D20: SB140, Diode_THT:D_DO-41_SOD81_P10.16mm_Horizontal, F.Cu at (79.8, 127.3)
- added D23: SB140, Diode_THT:D_DO-41_SOD81_P10.16mm_Horizontal, F.Cu at (107.4, 128.3)
- added D24: SB140, Diode_THT:D_DO-41_SOD81_P10.16mm_Horizontal, F.Cu at (115.6, 138.4)
- moved C57 1.78 mm to (173.0, 128.8)
Connections:
- C50 pad 1: GND -> LDRIVE+
- C50 pad 2: LDRIVE+ -> GND
- C52 pad 1: GND -> LDRIVE+
- C52 pad 2: LDRIVE+ -> GND
- C54 pad 1: GND -> RDRIVE+
- C54 pad 2: RDRIVE+ -> GND
- C56 pad 1: GND -> RDRIVE+
- C56 pad 2: RDRIVE+ -> GND
- U11 pad 5: (no net) -> GND
- U11 pad 6: (no net) -> Net-(U11B--)
- U11 pad 7: (no net) -> Net-(U11B--)
- U2 pad 5: (no net) -> GND
- U2 pad 6: (no net) -> Net-(U2B--)
- U2 pad 7: (no net) -> Net-(U2B--)
- U9 pad 5: (no net) -> GND
- U9 pad 6: (no net) -> Net-(U9B--)
- U9 pad 7: (no net) -> Net-(U9B--)
Routing:
- net +5V: track 346.4 -> 411.2 mm
- net Net-(D19-A): track 27.5 -> 87.3 mm
- net Net-(D23-A): track 41.4 -> 77.2 mm
- net Net-(D15-A): track 35.1 -> 65.3 mm
- net Net-(D17-A): track 46.2 -> 71.3 mm
- net GND: track 0.13 -> 6.89 mm, vias 53 -> 54
- net Net-(U2B--): track 0.00 -> 2.54 mm
- net Net-(U9B--): track 0.00 -> 2.54 mm
- net Net-(U11B--): track 0.00 -> 2.54 mm
- net LPWR+: track 160.6 -> 162.2 mm
- net BIAS: track 346.8 -> 348.3 mm
- net Net-(Q10-S): track 156.9 -> 158.2 mm
- net Net-(Q1-S): track 171.5 -> 172.6 mm
- net RPWR+: track 89.0 -> 88.2 mm
- net RDRIVE+: track 146.6 -> 146.0 mm
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Other:
- board text added: "Rev 1.1 https://github.com/prydin/classd-amp"
