File: left.kicad_sch (KiCad schematic)
At the start: 52 parts

Commit message: First prototype
Parts:
- added J1: LEFT, TerminalBlock_4Ucon:TerminalBlock_4Ucon_1x02_P3.50mm_Horizontal, symbol Connector:Screw_Terminal_01x02
Connections:
- net LOUT+: now also J1.1 (Pin_1)
- net LOUT-: now also J1.2 (Pin_2)
Changed lines of the file:
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@@
     (stroke (width 0) (type default))
   )
-  (wire (pts (xy 273.05 67.31) (xy 273.05 77.47))
+  (wire (pts (xy 273.05 67.31) (xy 273.05 88.9))
     (stroke (width 0) (type default))
   )
@@
     (stroke (width 0) (type default))
   )
-  (wire (pts (xy 273.05 106.68) (xy 273.05 132.08))
+  (wire (pts (xy 273.05 91.44) (xy 273.05 132.08))
     (stroke (width 0) (type default))
   )
@@
         )
       )
+    )
+  )
+  (symbol (lib_id "Connector:Screw_Terminal_01x02") (at 278.13 88.9 0) (unit 1)
+    (in_bom yes) (on_board yes) (dnp no) (fields_autoplaced)
+    (property "Reference" "J1" (at 280.67 88.9 0)
+      (effects (font (size 1.27 1.27)) (justify left))
+    )
+    (property "Value" "LEFT" (at 280.67 91.44 0)
+      (effects (font (size 1.27 1.27)) (justify left))
+    )
+    (property "Footprint" "TerminalBlock_4Ucon:TerminalBlock_4Ucon_1x02_P3.50mm_Horizontal" (at 278.13 88.9 0)
+      (effects (font (size 1.27 1.27)) hide)
+    )
+    (property "Datasheet" "~" (at 278.13 88.9 0)
+      (effects (font (size 1.27 1.27)) hide)
+    )
+    (pin "1")
+    (pin "2")
+    (instances
+      (project "classd-amp"
+        (path "/4342a3a3-4383-4661-90ac-821979f46c8c/3b3caeaf-3878-4281-86ae-73a7190e5fd4"
+          (reference "J1") (unit 1)
+        )
+        (path "/4342a3a3-4383-4661-90ac-821979f46c8c/2cb4c6d9-a527-4110-8e74-588e462bfe69"
+          (reference "J3") (unit 1)
+        )
+      )

Commit message: Pre layer elimination
Parts:
- added C58: 220p, Capacitor_THT:C_Disc_D3.4mm_W2.1mm_P2.50mm, symbol Device:C
- added C? (x2): 10u, Capacitor_THT:CP_Radial_D5.0mm_P2.50mm, symbol Device:C_Polarized
- added C? (x2): 100n, Capacitor_THT:C_Disc_D3.4mm_W2.1mm_P2.50mm, symbol Device:C
- added R41: 10k, Resistor_THT:R_Axial_DIN0204_L3.6mm_D1.6mm_P7.62mm_Horizontal, symbol Device:R
- C? (x2): value 10u -> 470n; footprint Capacitor_THT:CP_Radial_D4.0mm_P1.50mm -> Capacitor_THT:C_Rect_L9.0mm_W3.8mm_P7.50mm_MKT; symbol Device:C_Polarized -> Device:C
- RV?: value 1k -> 2k
Connections:
- net DRIVE+: now also C?.1, C?.1, C?.2, C?.2
- net GND: now also C58.2, C?.1, C?.1, C?.2, C?.2
- net LIN: now also C58.1, R41.2; no longer C?.2
- net at RV?.1: now also C?.2; no longer C?.1
- net at C?.1, D?.1 (K), U?.8 (VB): no longer D?.1 (K), R?.1, U?.7 (HO)
- new net: D?.1 (K), R?.1, U?.7 (HO)
- new net: C?.1, R41.1
Other:
- moved on the sheet: C?, Q?, R?

Commit message: WIP
Parts:
- added C60: 4.7n, Capacitor_THT:C_Disc_D3.4mm_W2.1mm_P2.50mm, symbol Device:C
- added C61, C62: 220p, Capacitor_THT:C_Disc_D3.4mm_W2.1mm_P2.50mm, symbol Device:C
- C58: value 220p -> 4.7n
- D? (x2): value 1N4001 -> MUR460
Connections:
- net BIAS: now also C61.1, C62.1
- net GND: now also C60.2, C61.2, C62.2
- net LIN: no longer C58.1
- net at C?.2, C?.2, RV?.2: now also C58.1
- net at C?.1, R41.1: now also C60.1
- net DRIVE+ renamed LDRIVE+
Other:
- moved on the sheet: D?, L?, R?

Commit message: Ver 1.1
Parts:
- added D? (x4): SB140, Diode_THT:D_DO-41_SOD81_P10.16mm_Horizontal, symbol Device:D_Schottky
- added U2: TL072, PCM_Package_DIP_AKL:DIP-8_W7.62mm, symbol Amplifier_Operational:TL072
Connections:
- net +5V: now also D?.1 (K), D?.1 (K)
- net GND: now also C?.2, C?.2, D?.2 (A), D?.2 (A), U2.5 (+); no longer C?.1, C?.1
- net LDRIVE+: now also C?.1, C?.1; no longer C?.2, C?.2
- net at C?.1, C?.1, R?.1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: now also D?.1 (K), D?.2 (A)
- net at C?.1, R?.1, R?.2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: now also D?.1 (K), D?.2 (A)
- new net: U2.6 (-), U2.7

Commit message: WIP
Parts:
- L? (x2): value 33u -> 22u
Changed lines of the file:
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@@
       (effects (font (size 1.27 1.27)))
     )
-    (property "Value" "33u" (at 255.27 128.905 90)
+    (property "Value" "22u" (at 255.27 128.905 90)
       (effects (font (size 1.27 1.27)))
     )
@@
       (effects (font (size 1.27 1.27)))
     )
-    (property "Value" "33u" (at 256.54 62.865 90)
-      (effects (font (size 1.27 1.27)))
-    )
+    (property "Value" "22u" (at 256.54 62.865 90)
+      (effects (font (size 1.27 1.27)))
+    )

Commit message: WIP
Parts:
- gave numbers to parts that had none: 59
- renumbered J1 to J3

Commit message: WIP
Parts:
- C1, C2, C4, C5, C6: footprint Capacitor_THT:CP_Radial_D8.0mm_P3.50mm -> Capacitor_THT:CP_Radial_D4.0mm_P1.50mm
- U1, U2, U4, U5, U6: footprint PCM_Package_DIP_AKL:DIP-8_W7.62mm -> Package_DIP:DIP-8_W7.62mm
Connections:
- net +5V: no longer D15.1 (K), D17.1 (K)
- net GND: now also D15.2 (A); no longer D16.2 (A)
- net LDRIVE+: now also D16.1 (K), D17.1 (K)
- net at C15.2, L2.1, Q1.3 (S)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: now also D15.1 (K), D16.2 (A)
- net at C16.1, D2.1 (K), U6.8 (VB): now also D5.1 (K), R11.1, U6.7 (HO)
- net at C10.1, C8.1, R5.2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: no longer D17.2 (A), D18.1 (K)
- net at C9.1, R6.2, R8.1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: no longer D15.2 (A), D16.1 (K)
- new net: D17.2 (A), D18.1 (K)
Other:
- moved on the sheet: C22, C50, C51, C52, C53, D3, D4, D5, D6, L2, Q1, Q2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
