File: right.kicad_sch (KiCad schematic)
At the start: 64 parts, among them J4 RIGHT, Q10 IRF540N, Q11 IRF540N, Q8 IRF540N, Q9 IRF540N, U10 TL072, U11 TL072, U12 LT1016, U13 IR2184, U14 IR2184

Commit message: WIP
Parts:
- D19, D20, D23, D24: footprint Diode_THT:D_DO-41_SOD81_P10.16mm_Horizontal -> Diode_THT:D_DO-41_SOD81_P5.08mm_Vertical_KathodeUp
- U10, U11, U12, U13, U14: footprint PCM_Package_DIP_AKL:DIP-8_W7.62mm -> Package_DIP:DIP-8_W7.62mm
- U11: footprint (none) -> Package_DIP:DIP-8_W7.62mm
Changed lines of the file:
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@@
 			)
 		)
-		(property "Footprint" ""
+		(property "Footprint" "Package_DIP:DIP-8_W7.62mm"
 			(at 102.87 144.145 0)
 			(effects
@@
 			)
 		)
-		(property "Footprint" "PCM_Package_DIP_AKL:DIP-8_W7.62mm"
+		(property "Footprint" "Package_DIP:DIP-8_W7.62mm"
 			(at 64.77 63.5 0)
 			(effects
@@
 			)
 		)
-		(property "Footprint" "Diode_THT:D_DO-41_SOD81_P10.16mm_Horizontal"
+		(property "Footprint" "Diode_THT:D_DO-41_SOD81_P5.08mm_Vertical_KathodeUp"
 			(at 107.95 118.745 0)
 			(effects
@@
 			)
 		)
-		(property "Footprint" "PCM_Package_DIP_AKL:DIP-8_W7.62mm"
+		(property "Footprint" "Package_DIP:DIP-8_W7.62mm"
 			(at 185.42 66.04 0)
 			(effects
@@
 			)
 		)
-		(property "Footprint" "Diode_THT:D_DO-41_SOD81_P10.16mm_Horizontal"
+		(property "Footprint" "Diode_THT:D_DO-41_SOD81_P5.08mm_Vertical_KathodeUp"
 			(at 81.28 41.91 0)
 			(effects
@@
 			)
 		)
-		(property "Footprint" "PCM_Package_DIP_AKL:DIP-8_W7.62mm"
+		(property "Footprint" "Package_DIP:DIP-8_W7.62mm"
 			(at 120.65 66.04 0)
 			(effects
@@
 			)
 		)
-		(property "Footprint" "Diode_THT:D_DO-41_SOD81_P10.16mm_Horizontal"
+		(property "Footprint" "Diode_THT:D_DO-41_SOD81_P5.08mm_Vertical_KathodeUp"
 			(at 81.28 29.21 0)
 			(effects
@@
 			)
 		)
-		(property "Footprint" "PCM_Package_DIP_AKL:DIP-8_W7.62mm"
+		(property "Footprint" "Package_DIP:DIP-8_W7.62mm"
 			(at 66.04 110.49 0)
 			(effects
@@
 			)
 		)
-		(property "Footprint" "PCM_Package_DIP_AKL:DIP-8_W7.62mm"
+		(property "Footprint" "Package_DIP:DIP-8_W7.62mm"
 			(at 185.42 132.08 0)
 			(effects
@@
 			)
 		)
-		(property "Footprint" "PCM_Package_DIP_AKL:DIP-8_W7.62mm"
+		(property "Footprint" "Package_DIP:DIP-8_W7.62mm"
 			(at 149.86 68.58 0)
 			(effects
@@
 			)
 		)
-		(property "Footprint" "Diode_THT:D_DO-41_SOD81_P10.16mm_Horizontal"
+		(property "Footprint" "Diode_THT:D_DO-41_SOD81_P5.08mm_Vertical_KathodeUp"
 			(at 107.95 102.87 0)
 			(effects
