File: right.kicad_sch (KiCad schematic)
At the start: 52 parts

Commit message: First prototype
Parts:
- added J1: RIGHT, TerminalBlock_4Ucon:TerminalBlock_4Ucon_1x02_P3.50mm_Horizontal, symbol Connector:Screw_Terminal_01x02
Connections:
- net ROUT+: now also J1.1 (Pin_1)
- net ROUT-: now also J1.2 (Pin_2)
Changed lines of the file:
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@@
     (stroke (width 0) (type default))
   )
-  (wire (pts (xy 273.05 67.31) (xy 273.05 77.47))
+  (wire (pts (xy 273.05 67.31) (xy 273.05 95.25))
     (stroke (width 0) (type default))
   )
@@
     (stroke (width 0) (type default))
   )
-  (wire (pts (xy 273.05 106.68) (xy 273.05 132.08))
-    (stroke (width 0) (type default))
-  )
   (wire (pts (xy 201.93 58.42) (xy 201.93 62.23))
     (stroke (width 0) (type default))
@@
   )
   (wire (pts (xy 157.48 71.12) (xy 168.91 71.12))
+    (stroke (width 0) (type default))
+  )
+  (wire (pts (xy 273.05 97.79) (xy 273.05 132.08))
     (stroke (width 0) (type default))
   )
@@
     (effects (font (size 1.27 1.27)) (justify left bottom))
   )
-  (label "ROUT-" (at 273.05 106.68 0) (fields_autoplaced)
+  (label "ROUT-" (at 273.05 114.3 0) (fields_autoplaced)
     (effects (font (size 1.27 1.27)) (justify left bottom))
   )
@@
         )
         (path "/4342a3a3-4383-4661-90ac-821979f46c8c/20bf2a2d-17c0-47aa-a67f-2d21b1e12aea"
-          (reference "RV1") (unit 2)
+          (reference "RV3") (unit 1)
         )
       )
@@
         )
       )
+    )
+  )
+  (symbol (lib_id "Connector:Screw_Terminal_01x02") (at 278.13 95.25 0) (unit 1)
+    (in_bom yes) (on_board yes) (dnp no) (fields_autoplaced)
+    (property "Reference" "J1" (at 280.67 95.25 0)
+      (effects (font (size 1.27 1.27)) (justify left))
+    )
+    (property "Value" "RIGHT" (at 280.67 97.79 0)
+      (effects (font (size 1.27 1.27)) (justify left))
+    )
+    (property "Footprint" "TerminalBlock_4Ucon:TerminalBlock_4Ucon_1x02_P3.50mm_Horizontal" (at 278.13 95.25 0)
+      (effects (font (size 1.27 1.27)) hide)
+    )
+    (property "Datasheet" "~" (at 278.13 95.25 0)
+      (effects (font (size 1.27 1.27)) hide)
+    )
+    (pin "1")
+    (pin "2")
+    (instances
+      (project "classd-amp"
+        (path "/4342a3a3-4383-4661-90ac-821979f46c8c/3b3caeaf-3878-4281-86ae-73a7190e5fd4"
+          (reference "J1") (unit 1)
+        )
+        (path "/4342a3a3-4383-4661-90ac-821979f46c8c/2cb4c6d9-a527-4110-8e74-588e462bfe69"
+          (reference "J3") (unit 1)
+        )
+        (path "/4342a3a3-4383-4661-90ac-821979f46c8c/20bf2a2d-17c0-47aa-a67f-2d21b1e12aea"
+          (reference "J4") (unit 1)
+        )
+      )

Commit message: Pre layer elimination
Parts:
- removed C?: 22u, Capacitor_THT:CP_Radial_D8.0mm_P3.50mm, symbol Device:C
- added C58: 220p, Capacitor_THT:C_Disc_D3.4mm_W2.1mm_P2.50mm, symbol Device:C
- added C? (x2): 10u, Capacitor_THT:CP_Radial_D5.0mm_P2.50mm, symbol Device:C_Polarized
- added C? (x2): 100n, Capacitor_THT:C_Disc_D3.4mm_W2.1mm_P2.50mm, symbol Device:C
- added C?: 22u, Capacitor_THT:CP_Radial_D8.0mm_P3.50mm, symbol Device:C
- added R41: 10k, Resistor_THT:R_Axial_DIN0204_L3.6mm_D1.6mm_P7.62mm_Horizontal, symbol Device:R
- C? (x2): value 10u -> 470n; footprint Capacitor_THT:CP_Radial_D4.0mm_P1.50mm -> Capacitor_THT:C_Rect_L9.0mm_W3.8mm_P7.50mm_MKT; symbol Device:C_Polarized -> Device:C
Connections:
- net DRIVE+: now also C?.1, C?.1, C?.2, C?.2
- net GND: now also C58.2, C?.1, C?.1, C?.2, C?.2
- net RIN: now also C58.1, R41.2
- net at RV?.1: now also C?.2
- net at C?.1, D?.1 (K), U?.8 (VB): no longer D?.1 (K), R?.1, U?.7 (HO)
- new net: C?.1, R41.1
- new net: D?.1 (K), R?.1, U?.7 (HO)
Other:
- moved on the sheet: Q?

Commit message: WIP
Parts:
- added C63, C64: 220p, Capacitor_THT:C_Disc_D3.4mm_W2.1mm_P2.50mm, symbol Device:C
Connections:
- net BIAS: now also C63.1, C64.1
- net GND: now also C63.2, C64.2
- net DRIVE+ renamed RDRIVE+
Changed lines of the file:
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@@
   (junction (at 57.15 66.04) (diameter 0) (color 0 0 0 0)
   )
+  (junction (at 57.15 43.815) (diameter 0) (color 0 0 0 0)
+  )
   (junction (at 238.76 82.55) (diameter 0) (color 0 0 0 0)
   )
+  (junction (at 135.89 71.12) (diameter 0) (color 0 0 0 0)
+  )
   (junction (at 232.41 127) (diameter 0) (color 0 0 0 0)
   )
@@
   (junction (at 124.46 36.83) (diameter 0) (color 0 0 0 0)
   )
+  (junction (at 49.53 43.815) (diameter 0) (color 0 0 0 0)
+  )
   (junction (at 273.05 67.31) (diameter 0) (color 0 0 0 0)
   )
@@
     (stroke (width 0) (type default))
   )
+  (wire (pts (xy 49.53 53.34) (xy 49.53 54.61))
+    (stroke (width 0) (type default))
+  )
   (wire (pts (xy 185.42 44.45) (xy 201.93 44.45))
     (stroke (width 0) (type default))
@@
     (stroke (width 0) (type default))
   )
+  (wire (pts (xy 49.53 43.18) (xy 49.53 43.815))
+    (stroke (width 0) (type default))
+  )
   (wire (pts (xy 33.02 69.85) (xy 33.02 72.39))
     (stroke (width 0) (type default))
@@
     (stroke (width 0) (type default))
   )
+  (wire (pts (xy 49.53 43.815) (xy 49.53 45.72))
+    (stroke (width 0) (type default))
+  )
   (wire (pts (xy 231.14 49.53) (xy 231.14 60.96))
     (stroke (width 0) (type default))
@@
     (stroke (width 0) (type default))
   )
+  (wire (pts (xy 125.095 71.12) (xy 135.89 71.12))
+    (stroke (width 0) (type default))
+  )
   (wire (pts (xy 259.08 143.51) (xy 259.08 156.21))
     (stroke (width 0) (type default))
@@
     (stroke (width 0) (type default))
   )
+  (wire (pts (xy 125.095 81.915) (xy 125.095 85.09))
+    (stroke (width 0) (type default))
+  )
   (wire (pts (xy 246.38 132.08) (xy 246.38 160.02))
     (stroke (width 0) (type default))
@@
     (stroke (width 0) (type default))
   )
-  (wire (pts (xy 57.15 53.34) (xy 57.15 60.96))
+  (wire (pts (xy 57.15 40.64) (xy 57.15 43.815))
     (stroke (width 0) (type default))
   )
@@
     (stroke (width 0) (type default))
   )
+  (wire (pts (xy 125.095 74.295) (xy 125.095 71.12))
+    (stroke (width 0) (type default))
+  )
   (wire (pts (xy 104.14 77.47) (xy 104.14 80.01))
     (stroke (width 0) (type default))
@@
     (stroke (width 0) (type default))
   )
+  (wire (pts (xy 49.53 43.815) (xy 57.15 43.815))
+    (stroke (width 0) (type default))
+  )
   (wire (pts (xy 227.33 116.84) (xy 232.41 116.84))
     (stroke (width 0) (type default))
@@
   )
   (wire (pts (xy 238.76 64.77) (xy 238.76 67.31))
+    (stroke (width 0) (type default))
+  )
+  (wire (pts (xy 57.15 43.815) (xy 57.15 60.96))
     (stroke (width 0) (type default))
   )
@@
     )
   )
-  (global_label "DRIVE+" (shape input) (at 238.76 48.26 90) (fields_autoplaced)
+  (global_label "RDRIVE+" (shape input) (at 238.76 48.26 90) (fields_autoplaced)
     (effects (font (size 1.27 1.27)) (justify left))
-    (property "Intersheetrefs" "${INTERSHEET_REFS}" (at 238.76 38.32 90)
+    (property "Intersheetrefs" "${INTERSHEET_REFS}" (at 238.76 37.05 90)
       (effects (font (size 1.27 1.27)) (justify left) hide)
     )
@@
     )
   )
-  (global_label "DRIVE+" (shape input) (at 240.03 113.03 90) (fields_autoplaced)
+  (global_label "RDRIVE+" (shape input) (at 240.03 113.03 90) (fields_autoplaced)
     (effects (font (size 1.27 1.27)) (justify left))
-    (property "Intersheetrefs" "${INTERSHEET_REFS}" (at 240.03 103.09 90)
+    (property "Intersheetrefs" "${INTERSHEET_REFS}" (at 240.03 101.82 90)
       (effects (font (size 1.27 1.27)) (justify left) hide)
     )
@@
     )
   )
-  (global_label "BIAS" (shape input) (at 57.15 53.34 90) (fields_autoplaced)
+  (global_label "BIAS" (shape input) (at 57.15 40.64 90) (fields_autoplaced)
     (effects (font (size 1.27 1.27)) (justify left))
-    (property "Intersheetrefs" "${INTERSHEET_REFS}" (at 57.15 46.1819 90)
+    (property "Intersheetrefs" "${INTERSHEET_REFS}" (at 57.15 33.4819 90)
       (effects (font (size 1.27 1.27)) (justify left) hide)
     )
@@
     )
   )
+  (symbol (lib_id "Device:C") (at 49.53 49.53 0) (unit 1)
+    (in_bom yes) (on_board yes) (dnp no) (fields_autoplaced)
+    (property "Reference" "C63" (at 52.705 48.26 0)
+      (effects (font (size 1.27 1.27)) (justify left))
+    )
+    (property "Value" "220p" (at 52.705 50.8 0)
+      (effects (font (size 1.27 1.27)) (justify left))
+    )
+    (property "Footprint" "Capacitor_THT:C_Disc_D3.4mm_W2.1mm_P2.50mm" (at 50.4952 53.34 0)
+      (effects (font (size 1.27 1.27)) hide)
+    )
+    (property "Datasheet" "~" (at 49.53 49.53 0)
+      (effects (font (size 1.27 1.27)) hide)
+    )
+    (pin "1")
+    (pin "2")
+    (instances
+      (project "classd-amp"
+        (path "/4342a3a3-4383-4661-90ac-821979f46c8c/20bf2a2d-17c0-47aa-a67f-2d21b1e12aea"
+          (reference "C63") (unit 1)
+        )
+      )
+    )
+  )
   (symbol (lib_id "Device:C") (at 175.26 116.84 0) (unit 1)
     (in_bom yes) (on_board yes) (dnp no) (fields_autoplaced)
@@
     )
   )
+  (symbol (lib_id "power:GND") (at 125.095 85.09 0) (unit 1)
+    (in_bom yes) (on_board yes) (dnp no) (fields_autoplaced)
+    (property "Reference" "#PWR064" (at 125.095 91.44 0)
+      (effects (font (size 1.27 1.27)) hide)
+    )
+    (property "Value" "GND" (at 125.095 90.17 0)
+      (effects (font (size 1.27 1.27)))
+    )
+    (property "Footprint" "" (at 125.095 85.09 0)
+      (effects (font (size 1.27 1.27)) hide)
+    )
+    (property "Datasheet" "" (at 125.095 85.09 0)
+      (effects (font (size 1.27 1.27)) hide)
+    )
+    (pin "1")
+    (instances
+      (project "classd-amp"
+        (path "/4342a3a3-4383-4661-90ac-821979f46c8c/20bf2a2d-17c0-47aa-a67f-2d21b1e12aea"
+          (reference "#PWR064") (unit 1)
+        )
+      )
+    )
+  )
   (symbol (lib_id "power:GND") (at 238.76 85.09 0) (unit 1)
     (in_bom yes) (on_board yes) (dnp no) (fields_autoplaced)
@@
         (path "/4342a3a3-4383-4661-90ac-821979f46c8c/20bf2a2d-17c0-47aa-a67f-2d21b1e12aea"
           (reference "#PWR049") (unit 1)
+        )
+      )
+    )
+  )
+  (symbol (lib_id "power:GND") (at 49.53 54.61 0) (unit 1)
+    (in_bom yes) (on_board yes) (dnp no) (fields_autoplaced)
+    (property "Reference" "#PWR063" (at 49.53 60.96 0)
+      (effects (font (size 1.27 1.27)) hide)
+    )
+    (property "Value" "GND" (at 49.53 59.69 0)
+      (effects (font (size 1.27 1.27)))
+    )
+    (property "Footprint" "" (at 49.53 54.61 0)
+      (effects (font (size 1.27 1.27)) hide)
+    )
+    (property "Datasheet" "" (at 49.53 54.61 0)
+      (effects (font (size 1.27 1.27)) hide)
+    )
+    (pin "1")
+    (instances
+      (project "classd-amp"
+        (path "/4342a3a3-4383-4661-90ac-821979f46c8c/20bf2a2d-17c0-47aa-a67f-2d21b1e12aea"
+          (reference "#PWR063") (unit 1)
         )
       )
@@
         )
       )
+    )
+  )
+  (symbol (lib_id "Device:C") (at 125.095 78.105 0) (unit 1)
+    (in_bom yes) (on_board yes) (dnp no) (fields_autoplaced)
+    (property "Reference" "C64" (at 128.27 76.835 0)
+      (effects (font (size 1.27 1.27)) (justify left))
+    )
+    (property "Value" "220p" (at 128.27 79.375 0)
+      (effects (font (size 1.27 1.27)) (justify left))
+    )
+    (property "Footprint" "Capacitor_THT:C_Disc_D3.4mm_W2.1mm_P2.50mm" (at 126.0602 81.915 0)
+      (effects (font (size 1.27 1.27)) hide)
+    )
+    (property "Datasheet" "~" (at 125.095 78.105 0)
+      (effects (font (size 1.27 1.27)) hide)
+    )
+    (pin "1")
+    (pin "2")
+    (instances
+      (project "classd-amp"
+        (path "/4342a3a3-4383-4661-90ac-821979f46c8c/20bf2a2d-17c0-47aa-a67f-2d21b1e12aea"
+          (reference "C64") (unit 1)
+        )
+      )

Commit message: Ver 1.1
Parts:
- added D? (x4): SB140, Diode_THT:D_DO-41_SOD81_P10.16mm_Horizontal, symbol Device:D_Schottky
- added U2: TL072, symbol Amplifier_Operational:TL072
Connections:
- net +5V: now also D?.1 (K), D?.1 (K)
- net GND: now also C?.2, C?.2, D?.2 (A), D?.2 (A), U2.5 (+); no longer C?.1, C?.1
- net RDRIVE+: now also C?.1, C?.1; no longer C?.2, C?.2
- net at C?.1, R?.1, R?.2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: now also D?.1 (K), D?.2 (A)
- net at C?.1, C?.1, R?.1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: now also D?.1 (K), D?.2 (A)
- new net: U2.6 (-), U2.7
Other:
- moved on the sheet: R?

Commit message: WIP
Parts:
- L? (x2): value 33u -> 22u
Changed lines of the file:
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@@
       (effects (font (size 1.27 1.27)))
     )
-    (property "Value" "33u" (at 255.27 128.905 90)
+    (property "Value" "22u" (at 255.27 128.905 90)
       (effects (font (size 1.27 1.27)))
     )
@@
       (effects (font (size 1.27 1.27)))
     )
-    (property "Value" "33u" (at 256.54 64.135 90)
-      (effects (font (size 1.27 1.27)))
-    )
+    (property "Value" "22u" (at 256.54 64.135 90)
+      (effects (font (size 1.27 1.27)))
+    )

Commit message: WIP
Parts:
- gave numbers to parts that had none: 59
- renumbered C58 to C18, J1 to J4, R41 to R42, U2 to U11

Commit message: Recovered PCB
Parts:
- renumbered C18 to C58, C54 to C?, C40 to C?, C43 to C?, C39 to C?, C45 to C?, C37 to C?, C20 to C?, C36 to C?, C19 to C?, C55 to C?, C41 to C?, C59 to C?, C47 to C?, C34 to C?, C33 to C?, C42 to C?, C46 to C?, C35 to C?, C57 to C?, C38 to C?, C44 to C?, C56 to C?, D20 to D?, D13 to D?, D24 to D?, D23 to D?, D8 to D?, D12 to D?, D9 to D?, D11 to D?, D19 to D?, D10 to D?, J4 to J1, L3 to L?, L4 to L?, Q10 to Q?, Q8 to Q?, Q11 to Q?, Q9 to Q?, R42 to R41, R31 to R?, R26 to R?, R30 to R?, R37 to R?, R29 to R?, R28 to R?, R33 to R?, R27 to R?, R36 to R?, R35 to R?, R38 to R?, R32 to R?, R39 to R?, R34 to R?, RV3 to RV?, RV4 to RV?, U11 to U2, U10 to U?, U13 to U?, U11 to U?, U14 to U?, U12 to U?
