File: power.kicad_sch (KiCad schematic)
At the start: 46 parts, among them J1 POWER, J5 POWER, Q12 2N3906, Q5 2N3906, Q6 2N3904, Q7 2N3904, U1 TL072, U10 TL072, U11 TL072, U2 TL072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

Commit message: Recovered PCB
Parts:
- removed C48, C49: 100n, Capacitor_THT:C_Disc_D3.4mm_W2.1mm_P2.50mm, symbol Device:C
- removed J5: POWER, TerminalBlock_4Ucon:TerminalBlock_4Ucon_1x02_P3.50mm_Horizontal, symbol Connector:Screw_Terminal_01x02
- removed Q12: 2N3906, Package_TO_SOT_THT:TO-92_Inline, symbol PCM_Transistor_BJT_AKL:2N3906
- removed R44: 1.5k, Resistor_THT:R_Axial_DIN0204_L3.6mm_D1.6mm_P7.62mm_Horizontal, symbol Device:R
- removed R45: 1k, Resistor_THT:R_Axial_DIN0204_L3.6mm_D1.6mm_P7.62mm_Horizontal, symbol Device:R
- removed R46: 4.7k, Resistor_THT:R_Axial_DIN0204_L3.6mm_D1.6mm_P7.62mm_Horizontal, symbol Device:R
- removed R47: 0.5, Resistor_THT:R_Axial_DIN0922_L20.0mm_D9.0mm_P25.40mm_Horizontal, symbol Device:R
- removed U10, U11: TL072, PCM_Package_DIP_AKL:DIP-8_W7.62mm, symbol Amplifier_Operational:TL072
- U1, U2, U9: footprint PCM_Package_DIP_AKL:DIP-8_W7.62mm -> Package_DIP:DIP-8_W7.62mm_LongPads
